File: camera-v3.0.sch (KiCad schematic (older format))
At the start: 9 parts, among them IC1 USB2660I-JZX-03, J1 1775862-2, J2 104031-0811, J3 503960-0696, J4 1-1734742-6, J5 1734742-8, U1 E73-2G4M08S1C-52840, U2 AXP209

Commit message: Мелкие фиксы
Parts:
- gave numbers to parts that had none: 1
Changed lines of the file:
@@
 $EndComp
 $Comp
-L mouser-local:53398-0867 J?
+L mouser-local:53398-0867 J6
 U 1 1 609EC819
 P 7100 7150
-F 0 "J?" H 7550 7415 50  0000 C CNN
+F 0 "J6" H 7550 7415 50  0000 C CNN
 F 1 "53398-0867" H 7550 7324 50  0000 C CNN
 F 2 "533980867" H 7850 7250 50  0001 L CNN
