File: camera-v3.0.kicad_pcb (KiCad board)
At the start: 2 copper layers, 60 x 39.8 mm, 7 parts, among them IC1 USB2660I-JZX-03, J1 1775862-2, J2 104031-0811, J3 503960-0696, U1 E73-2G4M08S1C-52840

Commit message: 111
Parts:
- removed J** (x2): 533980771, mouser-local:533980771
- added C1: 10u, mouser-local:CAPC3225X150N, F.Cu at (75.6, 47.4)
- added C10: 1u, mouser-local:CAPC1005X55N, F.Cu at (101.8, 36.5)
- added C11: 15n, mouser-local:CAPC1005X55N, F.Cu at (101.8, 34.5)
- added C12: 1u, mouser-local:CAPC1005X55N, F.Cu at (124.8, 45.3)
- added C13: 16p, mouser-local:CAPC1005X55N, F.Cu at (131.0, 38.8)
- added C14: 16p, mouser-local:CAPC1005X55N, F.Cu at (128.2, 43.1)
- added C15: 16p, mouser-local:CAPC1005X55N, F.Cu at (131.0, 40.8)
- added C16: 0.1u, mouser-local:CAPC1005X55N, F.Cu at (124.8, 47.3)
- added C17: 22u, mouser-local:CAPC3225X270N, F.Cu at (113.9, 45.1)
- added C18: 22u, mouser-local:CAPC3225X270N, F.Cu at (124.2, 35.6)
- added C19: 22u, mouser-local:CAPC3225X270N, F.Cu at (113.9, 41.0)
- added C2: 10u, mouser-local:CAPC3225X150N, F.Cu at (97.7, 39.6)
- added C20: 22u, mouser-local:CAPC3225X270N, F.Cu at (118.9, 35.6)
- added C21: 1u, mouser-local:CAPC1005X55N, F.Cu at (94.3, 63.3)
- added C22: 1u, mouser-local:CAPC1005X55N, F.Cu at (88.0, 67.7)
- added C23: 1u, mouser-local:CAPC1005X55N, F.Cu at (97.8, 58.9)
- added C24: 16p, mouser-local:CAPC1005X55N, F.Cu at (97.7, 61.0)
- added C25: 16p, mouser-local:CAPC1005X55N, F.Cu at (90.9, 67.7)
- added C26: 1u, mouser-local:CAPC1005X55N, F.Cu at (94.3, 65.3)
- added C27: 1u, mouser-local:CAPC1005X55N, F.Cu at (97.2, 63.3)
- added C28: 1u, mouser-local:CAPC1005X55N, F.Cu at (109.0, 54.6)
- added C3: 150p, mouser-local:CAPC1005X55N, F.Cu at (96.5, 44.8)
- added C4: 15n, mouser-local:CAPC1005X55N, F.Cu at (101.8, 38.5)
- added C5: 0.1u, mouser-local:CAPC1005X55N, F.Cu at (99.9, 42.7)
- added C6: 22u, mouser-local:CAPC3225X270N, F.Cu at (80.9, 47.4)
- added C7: 22u, mouser-local:CAPC3225X270N, F.Cu at (97.7, 35.6)
- added C8: 150p, mouser-local:CAPC1005X55N, F.Cu at (95.1, 47.6)
- added C9: 1u, mouser-local:CAPC1005X55N, F.Cu at (101.8, 40.4)
- added IC2: ADP1706ARDZ-3.3-R7, mouser-local:SOIC127P600X175-9N, F.Cu at (90.8, 36.8)
- added IC3: TUSB2046BVF, mouser-local:QFP80P900X900X160-32N, F.Cu at (78.7, 59.3)
- added IC4: GL823K, mouser-local:SOP64P600X175-16N, F.Cu at (88.7, 57.0)
- added J4: 73412-0110, mouser-local:73412-0110, B.Cu at (128.1, 103.5)
- added J5: 73412-0110, mouser-local:73412-0110, B.Cu at (127.9, 98.3)
- added L1: IHLP4040DZER6R8M01, mouser-local:INDPM108102X400N, F.Cu at (79.8, 39.5)
- added L2: 47n, mouser-local:LQW15CNR20J00B, F.Cu at (108.5, 46.3)
- added Q1: BC849B, mouser-local:SOT95P230X110-3N, F.Cu at (118.9, 39.9)
- added Q2: BC849B, mouser-local:SOT95P230X110-3N, F.Cu at (123.7, 39.9)
- added R1: 2k, mouser-local:RESC1005X40N, F.Cu at (92.0, 47.7)
- added R10: 4.7k, mouser-local:RESC1005X40N, F.Cu at (125.0, 43.2)
- added R11: 4.7k, mouser-local:RESC1005X40N, F.Cu at (121.6, 45.4)
- added R12: 4.7k, mouser-local:RESC1005X40N, F.Cu at (118.2, 45.4)
- added R13: 3k, mouser-local:RESC1005X40N, F.Cu at (128.5, 36.8)
- added R14: 10k, mouser-local:RESC1005X40N, F.Cu at (74.7, 66.2)
- added R15: 10k, mouser-local:RESC1005X40N, F.Cu at (81.5, 67.8)
- added R16: 1k5, mouser-local:RESC1005X40N, F.Cu at (94.6, 54.6)
- added R17: 10k, mouser-local:RESC1005X40N, F.Cu at (78.1, 66.2)
- added R18: 15k, mouser-local:RESC1005X40N, F.Cu at (74.7, 68.3)
- added R19: 15k, mouser-local:RESC1005X40N, F.Cu at (84.9, 67.8)
- added R2: 51.1, mouser-local:RESC1005X40N, F.Cu at (85.2, 47.7)
- added R20: 15k, mouser-local:RESC1005X40N, F.Cu at (94.6, 59.0)
- added R21: 15k, mouser-local:RESC1005X40N, F.Cu at (98.0, 56.8)
- added R22: 15k, mouser-local:RESC1005X40N, F.Cu at (94.6, 61.3)
- added R23: 15k, mouser-local:RESC1005X40N, F.Cu at (94.6, 56.8)
- added R24: 15k, mouser-local:RESC1005X40N, F.Cu at (98.0, 54.6)
- added R25: 15k, mouser-local:RESC1005X40N, F.Cu at (78.1, 68.3)
- added R26: 10k, mouser-local:RESC1005X40N, F.Cu at (105.9, 54.6)
- added R3: 30.1k, mouser-local:RESC1005X40N, F.Cu at (88.6, 47.7)
- added R4: 3k, mouser-local:RESC1005X40N, F.Cu at (96.8, 42.8)
- added R5: 22, mouser-local:RESC1005X40N, F.Cu at (128.5, 34.6)
- added R6: 22, mouser-local:RESC1005X40N, F.Cu at (121.6, 43.2)
- added R7: 22, mouser-local:RESC1005X40N, F.Cu at (127.8, 41.1)
- added R8: 4.7k, mouser-local:RESC1005X40N, F.Cu at (118.2, 43.2)
- added R9: 4.7k, mouser-local:RESC1005X40N, F.Cu at (127.8, 38.9)
- added U1: SIM7600E-H, SIM7600E-H:IC_SIM7600E-H, B.Cu at (98.4, 89.1)
- added Y1: 6MHz, mouser-local:ECS4802030BDUTR, F.Cu at (88.7, 63.5)
- IC1: value USB2660I-JZX-03 -> TPS54334DDA; footprint mouser:QFN50P900X900X100-65N-D -> mouser-local:SOIC127P600X170-9N
- J1: value 1775862-2 -> 104031-0811; footprint mouser:17758622 -> mouser-local:1040310811; moved to F.Cu
- J2: value 104031-0811 -> 503960-0696; footprint mouser:1040310811 -> mouser-local:5039600696
- J3: value 503960-0696 -> 73412-0110; footprint mouser:5039600696 -> mouser-local:73412-0110; moved to B.Cu
- moved IC1 47.1 mm to (90.8, 43.4)
- moved J3 36.9 mm to (127.9, 79.3), turned to 90 degrees
- moved J1 27.9 mm to (107.8, 104.6), turned to 0 degrees
- moved J2 21.1 mm to (90.9, 96.3)
- moved U2 0.92 mm to (118.1, 92.4)
- renumbered U1 to U2
Connections:
- net Net-(U1-Pad37) renamed SWDIO
- net Net-(U1-Pad39) renamed SWDCLK
- IC1 pad 1: Net-(IC1-Pad1) -> Net-(C5-Pad1)
- IC1 pad 2: Net-(IC1-Pad2) -> Vin
- IC1 pad 4: Net-(IC1-Pad4) -> GND
- J1 pad 1: Net-(J1-Pad1) -> SD_D2
- J1 pad 10: Net-(J1-Pad10) -> GND
- J1 pad 11: Net-(J1-Pad11) -> GND
- J1 pad 12: Net-(J1-Pad12) -> SD_CD
- J1 pad 13: Net-(J1-Pad13) -> GND
- J1 pad 14: Net-(J1-Pad14) -> GND
- J1 pad 2: Net-(J1-Pad2) -> SD_D3
- J1 pad 3: Net-(J1-Pad3) -> SD_CMD
- J1 pad 4: Net-(J1-Pad4) -> SD_POW
- J1 pad 5: Net-(J1-Pad5) -> SD_CLK
- J1 pad 6: Net-(J1-Pad6) -> GND
- J1 pad 7: Net-(J1-Pad7) -> SD_D0
- J1 pad 8: Net-(J1-Pad8) -> SD_D1
- J1 pad 9: Net-(J1-Pad9) -> GND
- U2 pad 19: Net-(U1-Pad19) -> +3V3
- U2 pad 21: Net-(U1-Pad21) -> GND
- U2 pad 24: Net-(U1-Pad24) -> GND
- U2 pad 29: Net-(IC1-Pad1) -> DM3
- U2 pad 31: Net-(IC1-Pad2) -> DP3
- U2 pad 5: Net-(U1-Pad5) -> GND
Other:
- outline, holes or cut-outs redrawn
