File: camera-v3.0.kicad_pcb (KiCad board)
At the start: 2 copper layers, 60 x 39.8 mm, 70 parts, among them IC1 TPS54334DDA, IC2 ADP1706ARDZ-3.3-R7, IC3 TUSB2046BVF, IC4 GL823K, J1 104031-0811, J2 503960-0696, J3 73412-0110, J4 73412-0110, J5 73412-0110, Q1 BC849B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

Commit message: Добавил разъемы
Parts:
- removed IC1: TPS54334DDA, mouser-local:SOIC127P600X170-9N
- removed IC2: ADP1706ARDZ-3.3-R7, mouser-local:SOIC127P600X175-9N
- removed IC3: TUSB2046BVF, mouser-local:QFP80P900X900X160-32N
- removed IC4: GL823K, mouser-local:SOP64P600X175-16N
- removed J1: 104031-0811, mouser-local:1040310811
- removed J2: 503960-0696, mouser-local:5039600696
- removed J3, J4, J5: 73412-0110, mouser-local:73412-0110
- added D1: TPS54334DDA, mouser-local:SOIC127P600X170-9N, F.Cu at (65.0, 65.3)
- added D2: ADP1706ARDZ-3.3-R7, mouser-local:SOIC127P600X175-9N, F.Cu at (56.5, 67.4)
- added D4: TUSB2046BVF, mouser-local:QFP80P900X900X160-32N, F.Cu at (61.2, 35.3)
- added D5: GL823K, mouser-local:SOP64P600X175-16N, F.Cu at (56.6, 44.5)
- added R27: 15k, mouser-local:RESC1005X40N, F.Cu at (54.0, 48.8)
- added R28: 15k, mouser-local:RESC1005X40N, F.Cu at (69.3, 41.5)
- added R29: 15k, mouser-local:RESC1005X40N, F.Cu at (72.1, 39.4)
- added R30: 15k, mouser-local:RESC1005X40N, F.Cu at (75.5, 37.2)
- added R31: 15k, mouser-local:RESC1005X40N, F.Cu at (65.9, 46.5)
- added R32: 10k, mouser-local:RESC1005X40N, F.Cu at (82.0, 56.0)
- added X1: 53398-0867, mouser-local:533980867, F.Cu at (129.4, 69.5)
- added X2: 1734742-8, mouser-local:17347428, F.Cu at (95.6, 69.4)
- added X3: SIM8065-6-1-14-01-A, mouser-local:SIM8065611401A, F.Cu at (95.4, 92.3)
- added X4: 73412-0110, mouser-local:73412-0110, F.Cu at (105.7, 32.1)
- added X5: 73412-0110, mouser-local:73412-0110, F.Cu at (100.7, 37.5)
- added X6: 73412-0110, mouser-local:73412-0110, F.Cu at (100.7, 32.1)
- added X7: 1-1734742-6, mouser-local:117347426, F.Cu at (110.0, 69.4)
- added X8: 104031-0811, mouser-local:1040310811, F.Cu at (105.6, 105.1)
- C12, C23: value 1u -> 16p
- C15: value 16p -> 0.1u
- C16: value 0.1u -> 22u; footprint mouser-local:CAPC1005X55N -> mouser-local:CAPC3225X270N
- C20: value 22u -> 1u; footprint mouser-local:CAPC3225X270N -> mouser-local:CAPC1005X55N
- C25: value 16p -> 1u
- R15, R17: value 10k -> DNP
- R16: value 1k5 -> DNP
- R18, R23: value 15k -> 10k
- R19: value 15k -> 1k5
- R20, R21, R22: value 15k -> DNP
- R26: value 10k -> 15k
- moved C20 66.9 mm to (53.8, 50.8)
- moved C7 56.7 mm to (54.9, 72.8)
- moved C10 55.4 mm to (59.0, 71.7)
- moved C4 49.2 mm to (59.1, 63.0)
- moved C21 47.6 mm to (53.8, 38.3)
- moved L1 46.0 mm to (45.5, 70.1)
- moved R26 45.4 mm to (60.8, 48.8)
- moved C11 43.1 mm to (73.6, 67.1)
- moved C23 41.9 mm to (56.6, 50.8)
- moved R13 40.4 mm to (89.9, 48.8)
- moved C3 39.6 mm to (67.5, 71.8)
- moved R1 39.3 mm to (62.6, 73.8)
- moved R3 39.3 mm to (59.2, 73.8)
- moved C22 38.8 mm to (76.8, 30.6)
- moved R11 38.7 mm to (83.1, 48.8)
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- renumbered U1 to D3, U2 to D6
Connections:
- C12 pad 1: SD_POW -> SIM_IO
- C13 pad 1: SIM_IO -> SIM_CLK
- C14 pad 1: SIM_CLK -> SIM_RST
- C15 pad 1: SIM_RST -> GND
- C15 pad 2: GND -> SIM_VCC
- C16 pad 1: GND -> +4V
- C16 pad 2: SIM_VCC -> GND
- C20 pad 1: +4V -> +3V3
- C23 pad 1: +3V3 -> Net-(C23-Pad1)
- C25 pad 1: Net-(C25-Pad1) -> +3V3
- C27 pad 1: +3V3 -> SD_POW
- D6 pad 26: Net-(R26-Pad1) -> Net-(D6-Pad26)
- R15 pad 1: GND -> SD_CLK
- R16 pad 1: +3V3 -> SD_D0
- R16 pad 2: CAM_DP -> Net-(R16-Pad2)
- R17 pad 1: Net-(IC3-Pad10) -> SD_D2
- R17 pad 2: +3V3 -> Net-(R17-Pad2)
- R18 pad 2: DP1 -> Net-(D4-Pad8)
- R19 pad 1: GND -> +3V3
- R19 pad 2: DM1 -> CAM_DP
- R20 pad 1: GND -> Net-(R20-Pad1)
- R20 pad 2: DP2 -> SD_CMD
- R21 pad 1: GND -> Net-(R21-Pad1)
- R21 pad 2: DM2 -> SD_D1
- R22 pad 1: GND -> Net-(R22-Pad1)
- R22 pad 2: DP3 -> SD_D3
- R23 pad 1: GND -> Net-(D4-Pad10)
- R23 pad 2: DM3 -> +3V3
- R24 pad 2: DP4 -> DP1
- R25 pad 2: DM4 -> DM1
- R26 pad 1: Net-(R26-Pad1) -> GND
- R26 pad 2: +3V3 -> DP2
- Y1 pad 1: Net-(C24-Pad1) -> Net-(C23-Pad1)
- Y1 pad 3: Net-(C25-Pad1) -> Net-(C24-Pad1)
