File: LTE.sch (KiCad schematic (older format))
At the start: 27 parts, among them J1 104031-0811, J2 503960-0696, J3 73412-0110, J4 73412-0110, J5 73412-0110, Q1 BC849B, Q2 BC849B, U1 SIM7600E-H

Commit message: Добавил разъемы
Parts:
- removed C12: 1u, CAPC1005X55N, symbol mouser-local:GRM155R61A105KE15J
- removed J1: 104031-0811, 1040310811, symbol mouser-local:104031-0811
- removed J2: 503960-0696, 5039600696, symbol camera-v3.0-rescue:503960-0696-mouser
- added X3: SIM8065-6-1-14-01-A, SIM8065611401A, symbol mouser-local:SIM8065-6-1-14-01-A
- renumbered C13 to C12, C14 to C13, C15 to C14, C16 to C15, C17 to C16, C18 to C17, C19 to C18, C20 to C19, U1 to D3, J3 to X4, J4 to X5, J5 to X6
Connections:
- net GND: now also X3.C5 (GND_1), X3.G1 (GND_2), X3.G2 (GND_3), X3.G3 (GND_4), X3.G4 (GND_5)
- net SIM_DET: now also X3.CD1 (CARD_DETECT)
- net SIM_VCC: now also X3.C1 (VCC)
- net at R5.2: now also X3.C2 (RST)
- net at R6.2: now also X3.C3 (CLK)
- net at R7.2: now also X3.C7 (I/O)
Other:
- moved on the sheet: C12, C13, C14, C15, R5, R6, R7
