File: NRF.sch (KiCad schematic (older format))
At the start: 3 parts, among them U2 E73-2G4M08S1C-52840

Commit message: Добавил разъемы
Parts:
- renumbered U2 to D6, R26 to R32
Changed lines of the file:
@@
 $EndDescr
 $Comp
-L nrfmicro:E73-2G4M08S1C-52840 U?
+L nrfmicro:E73-2G4M08S1C-52840 D?
 U 1 1 60E7E78C
 P 7500 4300
-AR Path="/60E7E78C" Ref="U?"  Part="1"
-AR Path="/611720F8/60E7E78C" Ref="U2"  Part="1"
-F 0 "U2" H 7475 5665 50  0000 C CNN
+AR Path="/60E7E78C" Ref="D?"  Part="1"
+AR Path="/611720F8/60E7E78C" Ref="D6"  Part="1"
+F 0 "D6" H 7475 5665 50  0000 C CNN
 F 1 "E73-2G4M08S1C-52840" H 7475 5574 50  0000 C CNN
 F 2 "nrfmicro:E73-2G4M08S1C-52840" H 7500 4300 50  0001 C CNN
@@
 AR Path="/60E94BE7" Ref="R?"  Part="1"
 AR Path="/6116F728/60E94BE7" Ref="R?"  Part="1"
-AR Path="/611720F8/60E94BE7" Ref="R26"  Part="1"
-F 0 "R26" H 8750 5100 50  0000 L CNN
+AR Path="/611720F8/60E94BE7" Ref="R32"  Part="1"
+F 0 "R32" H 8750 5100 50  0000 L CNN
 F 1 "10k" H 8850 5100 50  0000 L CNN
 F 2 "RESC1005X40N" H 9050 5050 50  0001 L CNN
@@
 AR Path="/60E96276" Ref="#PWR?"  Part="1"
 AR Path="/6116F728/60E96276" Ref="#PWR?"  Part="1"
-AR Path="/611720F8/60E96276" Ref="#PWR071"  Part="1"
-F 0 "#PWR071" H 9300 4850 50  0001 C CNN
+AR Path="/611720F8/60E96276" Ref="#PWR082"  Part="1"
+F 0 "#PWR082" H 9300 4850 50  0001 C CNN
 F 1 "+3.3V" H 9315 5173 50  0000 C CNN
 F 2 "" H 9300 5000 50  0001 C CNN
@@
 AR Path="/60E96DC2" Ref="#PWR?"  Part="1"
 AR Path="/6116F728/60E96DC2" Ref="#PWR?"  Part="1"
-AR Path="/611720F8/60E96DC2" Ref="#PWR070"  Part="1"
-F 0 "#PWR070" H 8600 4950 50  0001 C CNN
+AR Path="/611720F8/60E96DC2" Ref="#PWR081"  Part="1"
+F 0 "#PWR081" H 8600 4950 50  0001 C CNN
 F 1 "GND" H 8605 5027 50  0000 C CNN
 F 2 "" H 8600 5200 50  0001 C CNN
@@
 AR Path="/60E97628" Ref="#PWR?"  Part="1"
 AR Path="/6116F728/60E97628" Ref="#PWR?"  Part="1"
-AR Path="/611720F8/60E97628" Ref="#PWR067"  Part="1"
-F 0 "#PWR067" H 6250 4950 50  0001 C CNN
+AR Path="/611720F8/60E97628" Ref="#PWR078"  Part="1"
+F 0 "#PWR078" H 6250 4950 50  0001 C CNN
 F 1 "GND" H 6255 5027 50  0000 C CNN
 F 2 "" H 6250 5200 50  0001 C CNN
@@
 AR Path="/60E97C84" Ref="#PWR?"  Part="1"
 AR Path="/6116F728/60E97C84" Ref="#PWR?"  Part="1"
-AR Path="/611720F8/60E97C84" Ref="#PWR066"  Part="1"
-F 0 "#PWR066" H 6250 3350 50  0001 C CNN
+AR Path="/611720F8/60E97C84" Ref="#PWR077"  Part="1"
+F 0 "#PWR077" H 6250 3350 50  0001 C CNN
 F 1 "GND" H 6255 3427 50  0000 C CNN
 F 2 "" H 6250 3600 50  0001 C CNN
@@
 AR Path="/60E9A5C6" Ref="#PWR?"  Part="1"
 AR Path="/6116F728/60E9A5C6" Ref="#PWR?"  Part="1"
-AR Path="/611720F8/60E9A5C6" Ref="#PWR068"  Part="1"
-F 0 "#PWR068" H 6350 4850 50  0001 C CNN
+AR Path="/611720F8/60E9A5C6" Ref="#PWR079"  Part="1"
+F 0 "#PWR079" H 6350 4850 50  0001 C CNN
 F 1 "+3.3V" H 6365 5173 50  0000 C CNN
 F 2 "" H 6350 5000 50  0001 C CNN
@@
 AR Path="/60E9B2E6" Ref="#PWR?"  Part="1"
 AR Path="/6116F728/60E9B2E6" Ref="#PWR?"  Part="1"
-AR Path="/611720F8/60E9B2E6" Ref="#PWR069"  Part="1"
-F 0 "#PWR069" H 6450 5700 50  0001 C CNN
+AR Path="/611720F8/60E9B2E6" Ref="#PWR080"  Part="1"
+F 0 "#PWR080" H 6450 5700 50  0001 C CNN
 F 1 "GND" H 6455 5777 50  0000 C CNN
 F 2 "" H 6450 5950 50  0001 C CNN
@@
 Text GLabel 10150 3700 2    50   Input ~ 0
 LED_SCL
-Text GLabel 10150 3850 2    50   Input ~ 0
+Text GLabel 10150 3950 2    50   Input ~ 0
 BAT_SDA
-Text GLabel 10150 4000 2    50   Input ~ 0
+Text GLabel 10150 4100 2    50   Input ~ 0
 BAT_SCL
 $EndSCHEMATC
