File: POW.sch (KiCad schematic (older format))
At the start: 18 parts, among them IC1 TPS54334DDA, IC2 ADP1706ARDZ-3.3-R7

Commit message: Добавил разъемы
Parts:
- added X1: 53398-0867, 533980867, symbol mouser-local:53398-0867
- added X2: 1734742-8, 17347428, symbol mouser-local:1734742-8
- renumbered IC1 to D1, IC2 to D2
Connections:
- net +3V3: now also X2.3
- net GND: now also X1.4, X1.5, X1.6, X1.MP1, X1.MP2, X2.5, X2.6, X2.MP1, X2.MP2
- net Vin: now also X1.1, X1.2, X1.3, X2.8
- new net BAT_SCL: X1.7
- new net BAT_SDA: X1.8
- new net LED_PWM: X2.7
- new net LED_SCL: X2.1
- new net LED_SDA: X2.2
Changed lines of the file:
@@
 $EndDescr
 $Comp
-L mouser-local:TPS54334DDA IC1
+L mouser-local:TPS54334DDA D1
 U 1 1 60E2279F
 P 6300 3800
-F 0 "IC1" H 6850 4500 50  0000 C CNN
+F 0 "D1" H 6850 4500 50  0000 C CNN
 F 1 "TPS54334DDA" H 6900 4350 50  0000 C CNN
 F 2 "SOIC127P600X170-9N" H 7350 3900 50  0001 L CNN
@@
 $EndComp
 $Comp
-L power:GND #PWR03
+L power:GND #PWR010
 U 1 1 60E22815
 P 5850 5800
-F 0 "#PWR03" H 5850 5550 50  0001 C CNN
+F 0 "#PWR010" H 5850 5550 50  0001 C CNN
 F 1 "GND" H 5855 5627 50  0000 C CNN
 F 2 "" H 5850 5800 50  0001 C CNN
@@
 $EndComp
 $Comp
-L power:GND #PWR05
+L power:GND #PWR012
 U 1 1 60E2281B
 P 9450 4550
-F 0 "#PWR05" H 9450 4300 50  0001 C CNN
+F 0 "#PWR012" H 9450 4300 50  0001 C CNN
 F 1 "GND" H 9455 4377 50  0000 C CNN
 F 2 "" H 9450 4550 50  0001 C CNN
@@
 $EndComp
 $Comp
-L power:GND #PWR06
+L power:GND #PWR013
 U 1 1 60E22821
 P 9850 4550
-F 0 "#PWR06" H 9850 4300 50  0001 C CNN
+F 0 "#PWR013" H 9850 4300 50  0001 C CNN
 F 1 "GND" H 9855 4377 50  0000 C CNN
 F 2 "" H 9850 4550 50  0001 C CNN
@@
 Vin
 $Comp
-L power:GND #PWR02
+L power:GND #PWR09
 U 1 1 60E22836
 P 4800 4200
-F 0 "#PWR02" H 4800 3950 50  0001 C CNN
+F 0 "#PWR09" H 4800 3950 50  0001 C CNN
 F 1 "GND" H 4805 4027 50  0000 C CNN
 F 2 "" H 4800 4200 50  0001 C CNN
@@
 $EndComp
 $Comp
-L power:GND #PWR01
+L power:GND #PWR08
 U 1 1 60E2283C
 P 4300 4200
-F 0 "#PWR01" H 4300 3950 50  0001 C CNN
+F 0 "#PWR08" H 4300 3950 50  0001 C CNN
 F 1 "GND" H 4305 4027 50  0000 C CNN
 F 2 "" H 4300 4200 50  0001 C CNN
@@
 	4800 4150 4800 4200
 $Comp
-L power:GND #PWR04
+L power:GND #PWR011
 U 1 1 60E22844
 P 6200 4200
-F 0 "#PWR04" H 6200 3950 50  0001 C CNN
+F 0 "#PWR011" H 6200 3950 50  0001 C CNN
 F 1 "GND" H 6205 4027 50  0000 C CNN
 F 2 "" H 6200 4200 50  0001 C CNN
@@
 	10550 5700 10550 5800
 $Comp
-L power:GND #PWR07
+L power:GND #PWR014
 U 1 1 60E2289F
 P 10550 6600
-F 0 "#PWR07" H 10550 6350 50  0001 C CNN
+F 0 "#PWR014" H 10550 6350 50  0001 C CNN
 F 1 "GND" H 10555 6427 50  0000 C CNN
 F 2 "" H 10550 6600 50  0001 C CNN
@@
 	4800 3600 6300 3600
 $Comp
-L power:+4V #PWR08
+L power:+4V #PWR015
 U 1 1 60E228BC
 P 11400 3800
-F 0 "#PWR08" H 11400 3650 50  0001 C CNN
+F 0 "#PWR015" H 11400 3650 50  0001 C CNN
 F 1 "+4V" V 11415 3928 50  0000 L CNN
 F 2 "" H 11400 3800 50  0001 C CNN
@@
 $EndComp
 $Comp
-L mouser-local:ADP1706ARDZ-3.3-R7 IC2
+L mouser-local:ADP1706ARDZ-3.3-R7 D2
 U 1 1 60E228CA
 P 15150 3900
-F 0 "IC2" H 15750 4165 50  0000 C CNN
+F 0 "D2" H 15750 4165 50  0000 C CNN
 F 1 "ADP1706ARDZ-3.3-R7" H 15750 4074 50  0000 C CNN
 F 2 "SOIC127P600X175-9N" H 16200 4000 50  0001 L CNN
@@
 $EndComp
 $Comp
-L power:GND #PWR013
+L power:GND #PWR020
 U 1 1 60E228DE
 P 16550 4850
-F 0 "#PWR013" H 16550 4600 50  0001 C CNN
+F 0 "#PWR020" H 16550 4600 50  0001 C CNN
 F 1 "GND" H 16555 4677 50  0000 C CNN
 F 2 "" H 16550 4850 50  0001 C CNN
@@
 $EndComp
 $Comp
-L power:GND #PWR011
+L power:GND #PWR018
 U 1 1 60E228F3
 P 15050 4800
-F 0 "#PWR011" H 15050 4550 50  0001 C CNN
+F 0 "#PWR018" H 15050 4550 50  0001 C CNN
 F 1 "GND" H 15055 4627 50  0000 C CNN
 F 2 "" H 15050 4800 50  0001 C CNN
@@
 $EndComp
 $Comp
-L power:GND #PWR015
+L power:GND #PWR022
 U 1 1 60E22918
 P 17250 3900
-F 0 "#PWR015" H 17250 3650 50  0001 C CNN
+F 0 "#PWR022" H 17250 3650 50  0001 C CNN
 F 1 "GND" H 17255 3727 50  0000 C CNN
 F 2 "" H 17250 3900 50  0001 C CNN
@@
 	17100 3900 17250 3900
 $Comp
-L power:GND #PWR010
+L power:GND #PWR017
 U 1 1 60E22920
 P 14850 4000
-F 0 "#PWR010" H 14850 3750 50  0001 C CNN
+F 0 "#PWR017" H 14850 3750 50  0001 C CNN
 F 1 "GND" H 14855 3827 50  0000 C CNN
 F 2 "" H 14850 4000 50  0001 C CNN
@@
 	15150 4000 14850 4000
 $Comp
-L power:GND #PWR012
+L power:GND #PWR019
 U 1 1 60E22927
 P 15750 4800
-F 0 "#PWR012" H 15750 4550 50  0001 C CNN
+F 0 "#PWR019" H 15750 4550 50  0001 C CNN
 F 1 "GND" H 15755 4627 50  0000 C CNN
 F 2 "" H 15750 4800 50  0001 C CNN
@@
 	15050 4100 14450 4100
 $Comp
-L power:+4V #PWR09
+L power:+4V #PWR016
 U 1 1 60E2292F
 P 14450 4100
-F 0 "#PWR09" H 14450 3950 50  0001 C CNN
+F 0 "#PWR016" H 14450 3950 50  0001 C CNN
 F 1 "+4V" V 14465 4228 50  0000 L CNN
 F 2 "" H 14450 4100 50  0001 C CNN
@@
 $EndComp
 $Comp
-L power:+3.3V #PWR014
+L power:+3.3V #PWR021
 U 1 1 60E22935
 P 17000 4200
-F 0 "#PWR014" H 17000 4050 50  0001 C CNN
+F 0 "#PWR021" H 17000 4050 50  0001 C CNN
 F 1 "+3.3V" H 17015 4373 50  0000 C CNN
 F 2 "" H 17000 4200 50  0001 C CNN
@@
 Wire Wire Line
 	17000 4200 16550 4200
+$Comp
+L mouser-local:53398-0867 X1
+U 1 1 60EF6405
+P 3200 6000
+F 0 "X1" H 3650 6265 50  0000 C CNN
+F 1 "53398-0867" H 3650 6174 50  0000 C CNN
+F 2 "533980867" H 3950 6100 50  0001 L CNN
+F 3 "https://componentsearchengine.com/Datasheets/1/53398-0867.pdf" H 3950 6000 50  0001 L CNN
+F 4 "CONN WIRE TO BD HDR 8 POS 1.25MM SLDR ST SMD TAPE" H 3950 5900 50  0001 L CNN "Description"
+F 5 "5.9" H 3950 5800 50  0001 L CNN "Height"
+F 6 "Molex" H 3950 5700 50  0001 L CNN "Manufacturer_Name"
+F 7 "53398-0867" H 3950 5600 50  0001 L CNN "Manufacturer_Part_Number"
+F 8 "538-53398-0867" H 3950 5500 50  0001 L CNN "Mouser Part Number"
+F 9 "https://www.mouser.co.uk/ProductDetail/Molex/53398-0867?qs=d0WKAl%252BL4KZ2wnaw%2FdjEPw%3D%3D" H 3950 5400 50  0001 L CNN "Mouser Price/Stock"
+F 10 "" H 3950 5300 50  0001 L CNN "Arrow Part Number"
+F 11 "" H 3950 5200 50  0001 L CNN "Arrow Price/Stock"
+	1    3200 6000
+	1    0    0    -1
+$EndComp
+$Comp
+L power:GND #PWR01
+U 1 1 60EF8AFF
+P 2750 6400
+F 0 "#PWR01" H 2750 6150 50  0001 C CNN
+F 1 "GND" H 2755 6227 50  0000 C CNN
+F 2 "" H 2750 6400 50  0001 C CNN
+F 3 "" H 2750 6400 50  0001 C CNN
+	1    2750 6400
+	0    1    1    0
+$EndComp
+Text GLabel 4600 8000 2    50   Input ~ 0
+LED_SDA
+Text GLabel 2400 8000 0    50   Input ~ 0
+LED_SCL
+Text GLabel 2800 6000 0    50   Input ~ 0
+BAT_SDA
+Text GLabel 2800 6100 0    50   Input ~ 0
+BAT_SCL
+Text GLabel 2750 6700 0    50   Input ~ 0
+Vin
+$Comp
+L power:GND #PWR07
+U 1 1 60F002F6
+P 4250 6100
+F 0 "#PWR07" H 4250 5850 50  0001 C CNN
+F 1 "GND" H 4255 5927 50  0000 C CNN
+F 2 "" H 4250 6100 50  0001 C CNN
+F 3 "" H 4250 6100 50  0001 C CNN
+	1    4250 6100
+	0    -1   -1   0
+$EndComp
+Wire Wire Line
+	2800 6000 3200 6000
+Wire Wire Line
+	3200 6100 2800 6100
+Wire Wire Line
+	3200 6400 3000 6400
+Wire Wire Line
+	3200 6200 3000 6200
+Wire Wire Line
+	3000 6200 3000 6300
+Connection ~ 3000 6400
+Wire Wire Line
+	3000 6400 2750 6400
+Wire Wire Line
+	3200 6300 3000 6300
+Connection ~ 3000 6300
+Wire Wire Line
+	3000 6300 3000 6400
+Wire Wire Line
+	3200 6700 3000 6700
+Wire Wire Line
+	3200 6500 3000 6500
+Wire Wire Line
+	3000 6500 3000 6600
+Connection ~ 3000 6700
+Wire Wire Line
+	3000 6700 2750 6700
+Wire Wire Line
+	3200 6600 3000 6600
+Connection ~ 3000 6600
+Wire Wire Line
+	3000 6600 3000 6700
+Wire Wire Line
+	4100 6000 4150 6000
+Wire Wire Line
+	4150 6000 4150 6100
+Wire Wire Line
+	4150 6100 4250 6100
+Wire Wire Line
+	4100 6100 4150 6100
+Connection ~ 4150 6100
+Text GLabel 2400 8300 0    50   Input ~ 0
+LED_PWM
+$Comp
+L mouser-local:1734742-8 X2
+U 1 1 60F125F2
+P 3600 7700
+F 0 "X2" V 3600 7900 50  0000 C CNN
+F 1 "1734742-8" V 3700 8050 50  0000 C CNN
+F 2 "17347428" H 4450 8000 50  0001 L CNN
+F 3 "https://www.te.com/commerce/DocumentDelivery/DDEController?Action=showdoc&DocId=Customer+Drawing%7F1734742%7FP%7Fpdf%7FEnglish%7FENG_CD_1734742_P.pdf%7F1-1734742-8" H 4450 7900 50  0001 L CNN
+F 4 "TE Connectivity FPC 0.5mm Pitch 8 Way Straight SMT Female FPC Connector, ZIF Vertical Contact" H 4450 7800 50  0001 L CNN "Description"
+F 5 "5.3" H 4450 7700 50  0001 L CNN "Height"
+F 6 "TE Connectivity" H 4450 7600 50  0001 L CNN "Manufacturer_Name"
+F 7 "1734742-8" H 4450 7500 50  0001 L CNN "Manufacturer_Part_Number"
+F 8 "571-1734742-8" H 4450 7400 50  0001 L CNN "Mouser Part Number"
+F 9 "https://www.mouser.co.uk/ProductDetail/TE-Connectivity/1734742-8/?qs=n3Ybsy482HHYM%252Bd%2FbS4e5Q%3D%3D" H 4450 7300 50  0001 L CNN "Mouser Price/Stock"
+F 10 "1734742-8" H 4450 7200 50  0001 L CNN "Arrow Part Number"
+F 11 "https://www.arrow.com/en/products/1734742-8/te-connectivity" H 4450 7100 50  0001 L CNN "Arrow Price/Stock"
+	1    3600 7700
+	0    1    1    0
+$EndComp
+$Comp
+L power:+3.3V #PWR02
+U 1 1 60F155CF
+P 2750 8100
+F 0 "#PWR02" H 2750 7950 50  0001 C CNN
+F 1 "+3.3V" V 2750 8350 50  0000 C CNN
+F 2 "" H 2750 8100 50  0001 C CNN
+F 3 "" H 2750 8100 50  0001 C CNN
+	1    2750 8100
+	0    -1   -1   0
+$EndComp
+$Comp
+L power:GND #PWR06
+U 1 1 60F1738E
+P 4200 8200
+F 0 "#PWR06" H 4200 7950 50  0001 C CNN
+F 1 "GND" H 4205 8027 50  0000 C CNN
+F 2 "" H 4200 8200 50  0001 C CNN
+F 3 "" H 4200 8200 50  0001 C CNN
+	1    4200 8200
+	0    -1   -1   0
+$EndComp
+$Comp
+L power:GND #PWR03
+U 1 1 60F169FB
+P 2950 8200
+F 0 "#PWR03" H 2950 7950 50  0001 C CNN
+F 1 "GND" H 2955 8027 50  0000 C CNN
+F 2 "" H 2950 8200 50  0001 C CNN
+F 3 "" H 2950 8200 50  0001 C CNN
+	1    2950 8200
+	0    1    1    0
+$EndComp
+Text GLabel 4600 8300 2    50   Input ~ 0
+Vin
+$Comp
+L power:GND #PWR05
+U 1 1 60F1A036
+P 3600 8800
+F 0 "#PWR05" H 3600 8550 50  0001 C CNN
+F 1 "GND" H 3605 8627 50  0000 C CNN
+F 2 "" H 3600 8800 50  0001 C CNN
+F 3 "" H 3600 8800 50  0001 C CNN
+	1    3600 8800
+	1    0    0    -1
+$EndComp
+$Comp
+L power:GND #PWR04
+U 1 1 60F1A43B
+P 3600 7600
+F 0 "#PWR04" H 3600 7350 50  0001 C CNN
+F 1 "GND" H 3605 7427 50  0000 C CNN
+F 2 "" H 3600 7600 50  0001 C CNN
+F 3 "" H 3600 7600 50  0001 C CNN
+	1    3600 7600
+	-1   0    0    1
+$EndComp
+Wire Wire Line
+	3600 7700 3600 7600
+Wire Wire Line
+	3600 8700 3600 8800
+Wire Wire Line
+	4100 8200 4200 8200
+Wire Wire Line
+	4100 8300 4600 8300
+Wire Wire Line
+	4100 8000 4600 8000
+Wire Wire Line
+	2400 8000 3100 8000
+Wire Wire Line
+	3100 8100 2750 8100
+Wire Wire Line
+	2950 8200 3100 8200
+Wire Wire Line
+	3100 8300 2400 8300
 $EndSCHEMATC
