File: USB_HUB.sch (KiCad schematic (older format))
At the start: 22 parts, among them IC3 TUSB2046BVF, IC4 GL823K, Y1 6MHz

Commit message: Добавил разъемы
Parts:
- added C27: 1u, CAPC1005X55N, symbol mouser-local:GRM155R61A105KE15J
- added R15, R16, R17, R20, R21, R22: DNP, RESC1005X40N, symbol mouser-local:CRG0402F15R
- added X7: 1-1734742-6, 117347426, symbol mouser-local:1-1734742-6
- added X8: 104031-0811, 1040310811, symbol mouser-local:104031-0811
- renumbered C21 to C20, C22 to C21, C23 to C22, C24 to C23, C25 to C24, C26 to C25, C27 to C26, IC3 to D4, IC4 to D5, R15 to R18, R16 to R19, R17 to R23, R18 to R24, R19 to R25, R20 to R26, R21 to R27, R22 to R28, R23 to R29, R24 to R30, R25 to R31
Connections:
- net CAM_DM: now also X7.13
- net CAM_DP: now also X7.14
- net GND: now also C27.2, X7.11, X7.8, X7.MP1, X7.MP2, X8.10 (SH), X8.11 (SH), X8.13 (CD2), X8.14 (SH), X8.6 (VSS), X8.9 (SH)
- net SD_CD: now also X8.12 (CD1)
- net SD_CLK: now also R15.1, X8.5 (CLK)
- net SD_CMD: now also R20.2, X8.3 (CMD)
- net SD_D0: now also R16.1, X8.7 (DAT0)
- net SD_D1: now also R21.2, X8.8 (DAT1)
- net SD_D2: now also R17.1, X8.1 (DAT2)
- net SD_D3: now also R22.2, X8.2 (CD/DAT3)
- net SD_POW: now also C27.1, X8.4 (VDD)
- new net: R15.2, X7.1
- new net: R20.1, X7.2
- new net: R16.2, X7.3
- new net: R21.1, X7.4
- new net: R17.2, X7.5
- new net: R22.1, X7.6
